Commit message: Add mesh files and update inertial properties for camera URDF
- Added a new directory for meshes in setup.py to include necessary files.
- Updated the camera.urdf.xacro to reflect new mesh paths and corrected inertial properties for various components, including mass and inertia values for links such as base_link, servo, and others.

File: urdf/camera.urdf.xacro (robot description, xacro)
@@ -4,7 +4,7 @@
   <link name="base_link">
     <inertial>
-      <mass value="0.0"/>
-      <origin xyz="0.0 0.0 0.0" rpy="0.0 -0.0 0.0"/>
-      <inertia ixx="0.0" ixy="0.0" ixz="0.0" iyy="0.0" iyz="0.0" izz="0.0"/>
+      <mass value="0.05"/>
+      <origin xyz="0 0 0" rpy="0 0 0"/>
+      <inertia ixx="2e-4" ixy="0.0" ixz="0.0" iyy="2e-4" iyz="0.0" izz="2e-4"/>
     </inertial>
   </link>
@@ -14,5 +14,5 @@
       <origin xyz="0.0 0.02 0.02" rpy="0.0 -0.0 0.0"/>
       <geometry>
-        <mesh filename="package://camera/meshes/Camera_servo002.dae"/>
+        <mesh filename="package://yahboom_camera_controller/meshes/Camera_servo002.dae"/>
       </geometry>
     </visual>
@@ -21,11 +21,11 @@
       <origin xyz="0.0 0.02 0.02" rpy="0.0 -0.0 0.0"/>
       <geometry>
-        <mesh filename="package://camera/meshes/Camera_servo002.dae"/>
+        <mesh filename="package://yahboom_camera_controller/meshes/Camera_servo002.dae"/>
       </geometry>
     </collision>
     <inertial>
-      <mass value="0.0"/>
-      <origin xyz="0.0 0.0 0.0" rpy="0.0 -0.0 0.0"/>
-      <inertia ixx="0.0" ixy="0.0" ixz="0.0" iyy="0.0" iyz="0.0" izz="0.0"/>
+      <mass value="0.05"/>
+      <origin xyz="0 0 0" rpy="0 0 0"/>
+      <inertia ixx="1.8e-5" ixy="0.0" ixz="0.0" iyy="1.8e-5" iyz="0.0" izz="2.2e-5"/>
     </inertial>
   </link>
@@ -35,5 +35,5 @@
       <origin xyz="-0.01851 0.0125 -0.0135" rpy="0.0 -0.0 0.0"/>
       <geometry>
-        <mesh filename="package://camera/meshes/Camera_servo_mount001.dae"/>
+        <mesh filename="package://yahboom_camera_controller/meshes/Camera_servo_mount001.dae"/>
       </geometry>
     </visual>
@@ -42,11 +42,11 @@
       <origin xyz="-0.01851 0.0125 -0.0135" rpy="0.0 -0.0 0.0"/>
       <geometry>
-        <mesh filename="package://camera/meshes/Camera_servo_mount001.dae"/>
+        <mesh filename="package://yahboom_camera_controller/meshes/Camera_servo_mount001.dae"/>
       </geometry>
     </collision>
     <inertial>
-      <mass value="0.0"/>
-      <origin xyz="0.0 0.0 0.0" rpy="0.0 -0.0 0.0"/>
-      <inertia ixx="0.0" ixy="0.0" ixz="0.0" iyy="0.0" iyz="0.0" izz="0.0"/>
+      <mass value="0.03"/>
+      <origin xyz="0 0 0" rpy="0 0 0"/>
+      <inertia ixx="9e-6" ixy="0.0" ixz="0.0" iyy="9e-6" iyz="0.0" izz="1e-5"/>
     </inertial>
   </link>
@@ -56,5 +56,5 @@
       <origin xyz="-0.0185 0.0123 -0.0135" rpy="0.0 -0.0 0.0"/>
       <geometry>
-        <mesh filename="package://camera/meshes/Camera_bottom.dae"/>
+        <mesh filename="package://yahboom_camera_controller/meshes/Camera_bottom.dae"/>
       </geometry>
     </visual>
@@ -63,11 +63,11 @@
       <origin xyz="-0.0185 0.0123 -0.0135" rpy="0.0 -0.0 0.0"/>
       <geometry>
-        <mesh filename="package://camera/meshes/Camera_bottom.dae"/>
+        <mesh filename="package://yahboom_camera_controller/meshes/Camera_bottom.dae"/>
       </geometry>
     </collision>
     <inertial>
-      <mass value="0.0"/>
-      <origin xyz="0.0 0.0 0.0" rpy="0.0 -0.0 0.0"/>
-      <inertia ixx="0.0" ixy="0.0" ixz="0.0" iyy="0.0" iyz="0.0" izz="0.0"/>
+      <mass value="0.07"/>
+      <origin xyz="0 0 0" rpy="0 0 0"/>
+      <inertia ixx="3e-5" ixy="0.0" ixz="0.0" iyy="3e-5" iyz="0.0" izz="3.5e-5"/>
     </inertial>
   </link>
@@ -77,5 +77,5 @@
       <origin xyz="0.0 0.012 -0.04" rpy="0.0 -0.0 0.0"/>
       <geometry>
-        <mesh filename="package://camera/meshes/Camera_Connecting_rod.dae"/>
+        <mesh filename="package://yahboom_camera_controller/meshes/Camera_Connecting_rod.dae"/>
       </geometry>
     </visual>
@@ -84,11 +84,11 @@
       <origin xyz="0.0 0.012 -0.04" rpy="0.0 -0.0 0.0"/>
       <geometry>
-        <mesh filename="package://camera/meshes/Camera_Connecting_rod.dae"/>
+        <mesh filename="package://yahboom_camera_controller/meshes/Camera_Connecting_rod.dae"/>
       </geometry>
     </collision>
     <inertial>
-      <mass value="0.0"/>
-      <origin xyz="0.0 0.0 0.0" rpy="0.0 -0.0 0.0"/>
-      <inertia ixx="0.0" ixy="0.0" ixz="0.0" iyy="0.0" iyz="0.0" izz="0.0"/>
+      <mass value="0.02"/>
+      <origin xyz="0 0 0" rpy="0 0 0"/>
+      <inertia ixx="1.2e-6" ixy="0.0" ixz="0.0" iyy="1.2e-6" iyz="0.0" izz="1.3e-6"/>
     </inertial>
   </link>
@@ -98,5 +98,5 @@
       <origin xyz="0.041 -0.003 0.0" rpy="-0.0 -1.5707963267948961 0.0"/>
       <geometry>
-        <mesh filename="package://camera/meshes/Camera_top.dae"/>
+        <mesh filename="package://yahboom_camera_controller/meshes/Camera_top.dae"/>
       </geometry>
     </visual>
@@ -105,11 +105,11 @@
       <origin xyz="0.041 -0.003 0.0" rpy="-0.0 -1.5707963267948961 0.0"/>
       <geometry>
-        <mesh filename="package://camera/meshes/Camera_top.dae"/>
+        <mesh filename="package://yahboom_camera_controller/meshes/Camera_top.dae"/>
       </geometry>
     </collision>
     <inertial>
-      <mass value="0.0"/>
-      <origin xyz="0.0 0.0 0.0" rpy="0.0 -0.0 0.0"/>
-      <inertia ixx="0.0" ixy="0.0" ixz="0.0" iyy="0.0" iyz="0.0" izz="0.0"/>
+      <mass value="0.04"/>
+      <origin xyz="0 0 0" rpy="0 0 0"/>
+      <inertia ixx="1.6e-5" ixy="0.0" ixz="0.0" iyy="1.6e-5" iyz="0.0" izz="1.8e-5"/>
     </inertial>
   </link>
@@ -119,5 +119,5 @@
       <origin xyz="-0.019 -0.043 -0.037" rpy="0.0 -0.0 0.0"/>
       <geometry>
-        <mesh filename="package://camera/meshes/Camera_Lens.dae"/>
+        <mesh filename="package://yahboom_camera_controller/meshes/Camera_Lens.dae"/>
       </geometry>
     </visual>
@@ -126,11 +126,11 @@
       <origin xyz="-0.019 -0.043 -0.037" rpy="0.0 -0.0 0.0"/>
       <geometry>
-        <mesh filename="package://camera/meshes/Camera_Lens.dae"/>
+        <mesh filename="package://yahboom_camera_controller/meshes/Camera_Lens.dae"/>
       </geometry>
     </collision>
     <inertial>
-      <mass value="0.0"/>
-      <origin xyz="0.0 0.0 0.0" rpy="0.0 -0.0 0.0"/>
-      <inertia ixx="0.0" ixy="0.0" ixz="0.0" iyy="0.0" iyz="0.0" izz="0.0"/>
+      <mass value="0.01"/>
+      <origin xyz="0 0 0" rpy="0 0 0"/>
+      <inertia ixx="5e-7" ixy="0.0" ixz="0.0" iyy="5e-7" iyz="0.0" izz="6e-7"/>
     </inertial>
   </link>
